File: PCB/audio-amp-max98365.brd (EAGLE design)
At the start: 20 x 13 mm, 20 parts, among them U1 MAX98365

Commit message: Added BOM. Updated missing component values.
Parts:
- C1, C3: value (none) -> 1uF
- C2: value XXuF/xxV - 6.3mm -> 100uFuF/25V
- C4: value (none) -> 10uF
Changed lines of the file:
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@@
 <attribute name="NAME" x="16.355" y="1.285" size="1.016" layer="25" rot="R180" align="center-left"/>
 </element>
-<element name="C1" library="rlc" library_urn="urn:adsk.eagle:library:4192893" package="0603-CAP" package3d_urn="urn:adsk.eagle:package:4193021/2" value="" x="6.9" y="7.3" smashed="yes" rot="R180">
+<element name="C1" library="rlc" library_urn="urn:adsk.eagle:library:4192893" package="0603-CAP" package3d_urn="urn:adsk.eagle:package:4193021/2" value="1uF" x="6.9" y="7.3" smashed="yes" rot="R180">
 <attribute name="COST01" value="0.12" x="6.9" y="7.3" size="1.778" layer="27" rot="R180" display="off"/>
 <attribute name="COST10" value="0.09" x="6.9" y="7.3" size="1.778" layer="27" rot="R180" display="off"/>
@@
 <attribute name="VALUE" x="6.9" y="7.3" size="0.2" layer="27" rot="R180" align="center"/>
 </element>
-<element name="C2" library="rlc" library_urn="urn:adsk.eagle:library:4192893" package="CAP_ALUM_SMT_6.3" package3d_urn="urn:adsk.eagle:package:4192955/2" value="XXuF/xxV - 6.3mm" x="16.3" y="6.5" smashed="yes" rot="R90">
+<element name="C2" library="rlc" library_urn="urn:adsk.eagle:library:4192893" package="CAP_ALUM_SMT_6.3" package3d_urn="urn:adsk.eagle:package:4192955/2" value="100uFuF/25V" x="16.3" y="6.5" smashed="yes" rot="R90">
 <attribute name="NAME" x="14.69" y="2.975" size="0.9" layer="25" ratio="15" rot="R180"/>
 <attribute name="VALUE" x="20.145" y="3.475" size="0.4064" layer="27" rot="R90"/>
@@
 <attribute name="NAME" x="2.655" y="3.81" size="0.8128" layer="25" align="center-left"/>
 </element>
-<element name="C3" library="rlc" library_urn="urn:adsk.eagle:library:4192893" package="0603-CAP" package3d_urn="urn:adsk.eagle:package:4193021/2" value="" x="11.46" y="6" smashed="yes" rot="R180">
+<element name="C3" library="rlc" library_urn="urn:adsk.eagle:library:4192893" package="0603-CAP" package3d_urn="urn:adsk.eagle:package:4193021/2" value="1uF" x="11.46" y="6" smashed="yes" rot="R180">
 <attribute name="COST01" value="0.12" x="11.46" y="6" size="1.778" layer="27" rot="R180" display="off"/>
 <attribute name="COST10" value="0.09" x="11.46" y="6" size="1.778" layer="27" rot="R180" display="off"/>
@@
 <attribute name="VALUE" x="11.46" y="6" size="0.2" layer="27" rot="R180" align="center"/>
 </element>
-<element name="C4" library="rlc" library_urn="urn:adsk.eagle:library:4192893" package="0603-CAP" package3d_urn="urn:adsk.eagle:package:4193021/2" value="" x="11.46" y="7.3" smashed="yes" rot="R180">
+<element name="C4" library="rlc" library_urn="urn:adsk.eagle:library:4192893" package="0603-CAP" package3d_urn="urn:adsk.eagle:package:4193021/2" value="10uF" x="11.46" y="7.3" smashed="yes" rot="R180">
 <attribute name="COST01" value="0.12" x="11.46" y="7.3" size="1.778" layer="27" rot="R180" display="off"/>
 <attribute name="COST10" value="0.09" x="11.46" y="7.3" size="1.778" layer="27" rot="R180" display="off"/>
